Commit message: update README.md and finsih first version

File: bimanual/script/a5.urdf (robot description, URDF)
Before this commit: robot A5S, 7 links, 6 joints
Links:
- link link6: mass 0.58 -> 0.83

Commit message: update

File: bimanual/script/a5.urdf (robot description, URDF)
Before this commit: robot A5S, 7 links, 6 joints
Links:
- link link2: mass 0.882016949148399 -> 0.922016949148399
- link link6: mass 0.7 -> 0.68

Commit message: 必要更新 b535c1f

File: bimanual/script/a5.urdf (robot description, URDF)
Before this commit: robot A5S, 7 links, 6 joints
Links:
- link base_link: mass 0.42272 -> 0.652885471564488; geometry collision mesh filename=package://A5/meshes/base_link.STL; visual mesh filename=package://A5/meshes/base_link.STL
- link link1: mass 0.0968040209395549 -> 0.135332862135994; geometry collision mesh filename=package://A5/meshes/link1.STL; visual mesh filename=package://A5/meshes/link1.STL
- link link2: mass 0.922016949148399 -> 1.04903589366043; geometry collision mesh filename=package://A5/meshes/link2.STL; visual mesh filename=package://A5/meshes/link2.STL
- link link3: mass 0.887837614634739 -> 0.856398932000594; geometry collision mesh filename=package://A5/meshes/link3.STL; visual mesh filename=package://A5/meshes/link3.STL
- link link4: mass 0.118174840291438 -> 0.192580100804097; geometry collision mesh filename=package://A5/meshes/link4.STL; visual mesh filename=package://A5/meshes/link4.STL
- link link5: mass 0.636013398718114 -> 0.658983613915147; geometry collision mesh filename=package://A5/meshes/link5.STL; visual mesh filename=package://A5/meshes/link5.STL
- link link6: mass 0.68 -> 0.628913750332511; geometry collision mesh filename=package://A5/meshes/link6.STL; visual mesh filename=package://A5/meshes/link6.STL
Joints:
- joint joint1: origin xyz=0 0 0.0565 rpy=0 0 0 -> xyz=0 0 0.0695 rpy=0 0 0
- joint joint2: origin xyz=0.02 0 0.047 rpy=0 0 0 -> xyz=0.02 0 0.0435 rpy=0 0 0
- joint joint3: origin xyz=-0.21 -3E-05 0.06 rpy=0 0 0 -> xyz=-0.21 0 0.06 rpy=0 0 0
- joint joint4: origin xyz=0.189 -0.0001 0 rpy=-3.1416 0 0 -> xyz=0.189 0 0 rpy=3.1416 0 0
- joint joint5: origin xyz=0.07025 -5E-05 -0.0845 rpy=0 0 0 -> xyz=0.077 0 -0.0845 rpy=0 0 0
